Commit message: Fix URDF mesh paths and safety controller parameters, and remove broken tool joints

File: fairino_description/urdf/FR3WML.urdf (robot description, URDF)
Before this commit: robot FR3WML, 7 links, 7 joints
Links:
- link base_link: geometry collision mesh filename=package://fairino_description/meshes/FR3WML/collision/base_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; visual mesh filename=package://fairino_description/meshes/FR3WML/visual/base_lin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
- link forearm_Link: geometry collision mesh filename=package://fairino_description/meshes/FR3WML/collision/forea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; visual mesh filename=package://fairino_description/meshes/FR3WML/visual/forearm_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
- link shoulder_Link: geometry collision mesh filename=package://fairino_description/meshes/FR3WML/collision/shoul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; visual mesh filename=package://fairino_description/meshes/FR3WML/visual/shoulder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
- link upperarm_Link: geometry collision mesh filename=package://fairino_description/meshes/FR3WML/collision/upper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; visual mesh filename=package://fairino_description/meshes/FR3WML/visual/upperarm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
- link wrist1_Link: geometry collision mesh filename=package://fairino_description/meshes/FR3WML/collision/wrist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; visual mesh filename=package://fairino_description/meshes/FR3WML/visual/wrist1_L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
- link wrist2_Link: geometry collision mesh filename=package://fairino_description/meshes/FR3WML/collision/wrist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; visual mesh filename=package://fairino_description/meshes/FR3WML/visual/wrist2_L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
- link wrist3_Link: geometry collision mesh filename=package://fairino_description/meshes/FR3WML/collision/wrist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; visual mesh filename=package://fairino_description/meshes/FR3WML/visual/wrist3_L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
Joints:
- removed joint tool

File: fairino_description/urdf/FR3WMS.urdf (robot description, URDF)
Before this commit: robot FR3WMS, 7 links, 7 joints
Links:
- link base_link: geometry collision mesh filename=package://fairino_description/meshes/FR3WMS/collision/base_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; visual mesh filename=package://fairino_description/meshes/FR3WMS/visual/base_lin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
- link forearm_Link: geometry collision mesh filename=package://fairino_description/meshes/FR3WMS/collision/forea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; visual mesh filename=package://fairino_description/meshes/FR3WMS/visual/forearm_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
- link shoulder_Link: geometry collision mesh filename=package://fairino_description/meshes/FR3WMS/collision/shoul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; visual mesh filename=package://fairino_description/meshes/FR3WMS/visual/shoulder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
- link upperarm_Link: geometry collision mesh filename=package://fairino_description/meshes/FR3WMS/collision/upper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; visual mesh filename=package://fairino_description/meshes/FR3WMS/visual/upperarm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
- link wrist1_Link: geometry collision mesh filename=package://fairino_description/meshes/FR3WMS/collision/wrist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; visual mesh filename=package://fairino_description/meshes/FR3WMS/visual/wrist1_L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
- link wrist2_Link: geometry collision mesh filename=package://fairino_description/meshes/FR3WMS/collision/wrist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; visual mesh filename=package://fairino_description/meshes/FR3WMS/visual/wrist2_L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
- link wrist3_Link: geometry collision mesh filename=package://fairino_description/meshes/FR3WMS/collision/wrist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; visual mesh filename=package://fairino_description/meshes/FR3WMS/visual/wrist3_L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
Joints:
- removed joint tool
